File: org/lrn/apollo/apollo/apollo.kicad_pcb (KiCad board)
At the start: 2 copper layers, 47 parts, among them J1 Conn_01x01_Male, J2 Conn_01x01_Male, J3 Conn_01x01_Male, J4 Conn_01x01_Male, Q1 PN2222A, Q2 PN2222A, Q3 PN2222A, Q4 PN2222A, U1 74HC595, U2 5461AS-1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

Commit message: apollo: pcb optimizing
Parts:
- moved J_CLR1 106.4 mm to (239.3, 36.4)
- moved J_SER1 91.8 mm to (239.3, 42.2)
- moved J_CLK1 89.3 mm to (199.5, 48.0)
- moved J_GND1 4.87 mm to (193.8, 52.7)
Routing:
- net Net-(J_SER1-Pad1): track 124.7 -> 138.3 mm
- net Net-(J_CLK1-Pad1): track 145.5 -> 153.2 mm, vias 2 -> 3
- net GND: track 241.8 -> 248.6 mm
- net Net-(J_CLR1-Pad1): track 160.7 -> 155.5 mm
- net Net-(R1-Pad2): track 37.0 -> 40.0 mm
- net Net-(Q2-Pad3): track 17.9 -> 19.8 mm
- net Net-(J1-Pad1): track 23.0 -> 21.0 mm
- net Net-(J4-Pad1): track 20.7 -> 21.3 mm
