File: org/lrn/apollo/apollo/apollo.sch (KiCad schematic (older format))
At the start: 84 parts, among them J10 Conn_01x01_Male, J11 Conn_01x01_Male, J12 Conn_01x01_Male, J13 Conn_01x01_Male, J17 Conn_01x01_Male, J18 Conn_01x01_Male, J4 Conn_01x01_Male, J6 Conn_01x01_Male, J7 Conn_01x01_Male, J8 Conn_01x01_Male, J9 Conn_01x01_Male, Q1 PN2222A, Q2 PN2222A, Q3 PN2222A, Q4 PN2222A, Q5 PN2222A, Q6 PN2222A, U1 74HC595, U2 5461AS-1, U3 74HC595, U4 ATmega168P-20PU

Commit message: apollo: pcb compactification and optimization
Parts:
- removed J10, J11, JA_15, JB_1, JC_2, JD_3, JE_4, JF_5, JG_6, JH_1, JH_2, JH_3, JH_4, JH_7, JH_8: Conn_01x01_Male, Connector_Pin:Pin_D1.0mm_L10.0mm, symbol Connector:Conn_01x01_Male

Commit message: apollo: pcb compactify
Parts:
- removed JH_10, JH_11, JH_12, JH_13, JH_5, JH_6, JH_9: Conn_01x01_Male, Connector_Pin:Pin_D1.0mm_L10.0mm, symbol Connector:Conn_01x01_Male
Changed lines of the file:
@@
 	6400 4000 5300 4000
 Wire Wire Line
-	5300 4000 5300 4150
-Wire Wire Line
 	6400 4150 6650 4150
-$Comp
-L Connector:Conn_01x01_Male JH_5
-U 1 1 5F88F87C
-P 5900 4150
-F 0 "JH_5" H 6150 4100 50  0000 C CNN
-F 1 "Conn_01x01_Male" H 6150 4050 50  0000 C CNN
-F 2 "Connector_Pin:Pin_D1.0mm_L10.0mm" H 5900 4150 50  0001 C CNN
-F 3 "~" H 5900 4150 50  0001 C CNN
-	1    5900 4150
-	-1   0    0    1
-$EndComp
-$Comp
-L Connector:Conn_01x01_Male JH_6
-U 1 1 5F8C04F3
-P 5900 4350
-F 0 "JH_6" H 6100 4300 50  0000 C CNN
-F 1 "Conn_01x01_Male" H 6050 4400 50  0000 C CNN
-F 2 "Connector_Pin:Pin_D1.0mm_L10.0mm" H 5900 4350 50  0001 C CNN
-F 3 "~" H 5900 4350 50  0001 C CNN
-	1    5900 4350
-	-1   0    0    1
-$EndComp
 Wire Wire Line
 	6300 4650 6650 4650
@@
 	6300 4650 6300 4500
 Wire Wire Line
-	5400 4350 5400 4250
-Wire Wire Line
-	5400 4250 6400 4250
-Wire Wire Line
 	6400 4250 6400 4350
 Wire Wire Line
 	6400 4350 6650 4350
 Wire Wire Line
-	5300 4150 5700 4150
-Wire Wire Line
-	5400 4350 5700 4350
-Wire Wire Line
 	5500 4500 6300 4500
 Wire Wire Line
 	6300 4750 6300 5500
 Wire Wire Line
-	6300 5500 5600 5500
-Wire Wire Line
 	6300 4750 6650 4750
 Wire Wire Line
 	6300 5500 6850 5500
-Connection ~ 6300 5500
-$Comp
-L Connector:Conn_01x01_Male JH_10
-U 1 1 5FA1EBF7
-P 9050 1300
-F 0 "JH_10" H 8900 1300 50  0000 C CNN
-F 1 "Conn_01x01_Male" H 8400 1300 50  0000 C CNN
-F 2 "Connector_Pin:Pin_D1.0mm_L10.0mm" H 9050 1300 50  0001 C CNN
-F 3 "~" H 9050 1300 50  0001 C CNN
-	1    9050 1300
-	-1   0    0    1
-$EndComp
-$Comp
-L Connector:Conn_01x01_Male JH_11
-U 1 1 5FA2BDF0
-P 9050 1850
-F 0 "JH_11" H 8900 1850 50  0000 C CNN
-F 1 "Conn_01x01_Male" H 8400 1850 50  0000 C CNN
-F 2 "Connector_Pin:Pin_D1.0mm_L10.0mm" H 9050 1850 50  0001 C CNN
-F 3 "~" H 9050 1850 50  0001 C CNN
-	1    9050 1850
-	-1   0    0    1
-$EndComp
-$Comp
-L Connector:Conn_01x01_Male JH_12
-U 1 1 5FA39C16
-P 9050 2450
-F 0 "JH_12" H 8900 2450 50  0000 C CNN
-F 1 "Conn_01x01_Male" H 8400 2450 50  0000 C CNN
-F 2 "Connector_Pin:Pin_D1.0mm_L10.0mm" H 9050 2450 50  0001 C CNN
-F 3 "~" H 9050 2450 50  0001 C CNN
-	1    9050 2450
-	-1   0    0    1
-$EndComp
-$Comp
-L Connector:Conn_01x01_Male JH_13
-U 1 1 5FA4799A
-P 9050 3050
-F 0 "JH_13" H 8900 3050 50  0000 C CNN
-F 1 "Conn_01x01_Male" H 8400 3050 50  0000 C CNN
-F 2 "Connector_Pin:Pin_D1.0mm_L10.0mm" H 9050 3050 50  0001 C CNN
-F 3 "~" H 9050 3050 50  0001 C CNN
-	1    9050 3050
-	-1   0    0    1
-$EndComp
 $Comp
 L Transistor_BJT:PN2222A Q5
@@
 Wire Wire Line
 	5300 3100 5300 4000
-Connection ~ 5300 4000
 Wire Wire Line
 	1950 3200 5200 3200
 Wire Wire Line
 	5200 3200 5200 4250
-Wire Wire Line
-	5200 4250 5400 4250
-Connection ~ 5400 4250
 Wire Wire Line
 	1950 3500 2150 3500
@@
 	9500 2300 10050 2300
 Wire Wire Line
-	1950 2900 8750 2900
-Wire Wire Line
-	8850 1850 8750 1850
-Wire Wire Line
 	8750 1850 8750 1700
 Wire Wire Line
 	8750 1700 9200 1700
 Wire Wire Line
-	8850 2450 8750 2450
-Wire Wire Line
-	8750 2450 8750 2300
-Wire Wire Line
 	8750 2300 9200 2300
-Wire Wire Line
-	8850 3050 8750 3050
-Wire Wire Line
-	8750 3050 8750 2900
-Connection ~ 8750 2900
-Wire Wire Line
-	8750 2900 9200 2900
 Wire Wire Line
 	11100 600  11100 1400
@@
 Wire Wire Line
 	8750 1150 9200 1150
-Wire Wire Line
-	8750 1300 8850 1300
 Wire Wire Line
 	2000 4100 2000 5500
@@
 	7050 5500 7700 5500
 Wire Wire Line
-	5600 4750 5600 5500
-Wire Wire Line
-	5600 4750 5700 4750
-Wire Wire Line
 	1350 950  1350 1500
 Wire Wire Line
@@
 	1350 850  1350 950
 Wire Wire Line
-	8750 2800 8750 2450
-Connection ~ 8750 2450
-Wire Wire Line
 	1950 2800 8750 2800
 Wire Wire Line
@@
 Wire Wire Line
 	8650 1850 8750 1850
-Connection ~ 8750 1850
 Wire Wire Line
 	1950 2700 8650 2700
@@
 	10600 350  10600 -400
 Connection ~ 10600 -400
-Connection ~ 8750 1300
 Wire Wire Line
 	4900 2600 8550 2600
@@
 Wire Wire Line
 	7400 -150 8300 -150
-$Comp
-L Connector:Conn_01x01_Male JH_9
-U 1 1 5F970864
-P 5900 4750
-F 0 "JH_9" H 6100 4700 50  0000 C CNN
-F 1 "Conn_01x01_Male" H 6100 4950 50  0000 C CNN
-F 2 "Connector_Pin:Pin_D1.0mm_L10.0mm" H 5900 4750 50  0001 C CNN
-F 3 "~" H 5900 4750 50  0001 C CNN
-	1    5900 4750
-	-1   0    0    1
-$EndComp
+Wire Wire Line
+	1950 2900 9200 2900
+Wire Wire Line
+	8750 2300 8750 2800
+Wire Wire Line
+	5200 4250 6400 4250
 $EndSCHEMATC

Commit message: netlist optimization
Connections:
- net at U1.11 (SRCLK): now also U4.24 (PC1); no longer U4.28 (PC5)
- net at U1.14 (SER): now also U4.23 (PC0); no longer U4.27 (PC4)
- net at Rb1.2: now also U4.28 (PC5); no longer U4.26 (PC3)
- net at Rb2.2: now also U4.25 (PC2); no longer U4.23 (PC0)
- net at Rb3.2: now also U4.26 (PC3); no longer U4.24 (PC1)
- net at Rb4.2: now also U4.27 (PC4); no longer U4.25 (PC2)
Changed lines of the file:
@@
 	1350 950  3100 950
-Wire Wire Line
-	1950 3000 4900 3000
-Wire Wire Line
-	1950 3100 5300 3100
-Wire Wire Line
-	5300 3100 5300 4000
-Wire Wire Line
-	1950 3200 5200 3200
-Wire Wire Line
-	5200 3200 5200 4250
 Wire Wire Line
 	1950 3500 2150 3500
@@
 	9500 2300 10050 2300
 Wire Wire Line
-	8750 1850 8750 1700
-Wire Wire Line
-	8750 1700 9200 1700
-Wire Wire Line
 	8750 2300 9200 2300
 Wire Wire Line
@@
 Wire Wire Line
 	11100 1400 11100 1900
-Wire Wire Line
-	8750 1300 8750 1150
-Wire Wire Line
-	8750 1150 9200 1150
 Wire Wire Line
 	2000 4100 2000 5500
@@
 	1350 850  1350 950
 Wire Wire Line
-	1950 2800 8750 2800
-Wire Wire Line
-	8650 2700 8650 1850
-Wire Wire Line
-	8650 1850 8750 1850
-Wire Wire Line
-	1950 2700 8650 2700
-Wire Wire Line
-	4900 2600 4900 3000
-Wire Wire Line
 	4000 2200 4950 2200
 Wire Wire Line
@@
 	4900 2600 8550 2600
 Wire Wire Line
-	8550 1300 8750 1300
-Wire Wire Line
-	8550 2600 8550 1300
-Wire Wire Line
 	4850 -400 4850 -150
 Wire Wire Line
@@
 	7400 -150 8300 -150
 Wire Wire Line
-	1950 2900 9200 2900
-Wire Wire Line
 	8750 2300 8750 2800
 Wire Wire Line
 	5200 4250 6400 4250
+Wire Wire Line
+	1950 3200 4900 3200
+Wire Wire Line
+	4900 2600 4900 3200
+Wire Wire Line
+	1950 3100 4800 3100
+Wire Wire Line
+	4800 3100 4800 2900
+Wire Wire Line
+	4800 2900 9200 2900
+Wire Wire Line
+	1950 3000 4700 3000
+Wire Wire Line
+	4700 3000 4700 2800
+Wire Wire Line
+	4700 2800 8750 2800
+Wire Wire Line
+	1950 2900 4600 2900
+Wire Wire Line
+	4600 2900 4600 2700
+Wire Wire Line
+	4600 2700 8650 2700
+Wire Wire Line
+	8650 1700 9200 1700
+Wire Wire Line
+	8650 1700 8650 2700
+Wire Wire Line
+	8550 1150 8550 2600
+Wire Wire Line
+	8550 1150 9200 1150
+Wire Wire Line
+	1950 2800 4500 2800
+Wire Wire Line
+	4500 2800 4500 2400
+Wire Wire Line
+	4500 2400 5200 2400
+Wire Wire Line
+	5200 2400 5200 4250
+Wire Wire Line
+	1950 2700 4400 2700
+Wire Wire Line
+	4400 2700 4400 2300
+Wire Wire Line
+	4400 2300 5300 2300
+Wire Wire Line
+	5300 2300 5300 4000
 $EndSCHEMATC
